Commit message: Added Depth Camera robot.urdf

File: src/two_wheel_drive/urdf/robot.urdf (robot description, URDF)
Before this commit: robot two_wheel_robot, 7 links, 6 joints
Links:
- added link depth_camera_link; visual box size=0.01 0.01 0.01
- added link depth_camera_link_optical
Joints:
- added joint depth_camera_joint: type fixed, parent base_link, child depth_camera_link, origin xyz=0.155 0 0.02 rpy=0 0 0
- added joint depth_camera_joint_optical: type fixed, parent depth_camera_link, child depth_camera_link_optical, origin xyz=0 0 0 rpy=-1.5708 0 -1.5708

Commit message: Integrated autonav course Adjusted Robots size Increased camera height Correcteed spawn location

File: src/two_wheel_drive/urdf/robot.urdf (robot description, URDF)
Before this commit: robot two_wheel_robot, 9 links, 8 joints
Links:
- added link h_boom, mass 1.0; collision box size=0.02 0.02 0.5; visual box size=0.02 0.02 0.5
- link base_link: geometry collision box size=0.9 0.6 0.15; visual box size=0.9 0.6 0.15
- link caster: geometry collision sphere radius=0.06; visual sphere radius=0.06
- link depth_camera_link: geometry visual box size=0.03 0.03 0.03
- link gps_link: geometry collision cylinder length=0.06 radius=0.06; visual cylinder length=0.06 radius=0.06
- link imu_link: geometry collision box size=0.06 0.06 0.06; visual box size=0.06 0.06 0.06
- link left_wheel: geometry collision cylinder length=0.12 radius=0.15; visual cylinder length=0.12 radius=0.15
- link lidar_link: geometry collision cylinder length=0.06 radius=0.09; visual cylinder length=0.06 radius=0.09
- link right_wheel: geometry collision cylinder length=0.12 radius=0.15; visual cylinder length=0.12 radius=0.15
Joints:
- added joint h_boom_joint: type fixed, parent base_link, child h_boom, origin xyz=0 0 0.15 rpy=0 0 0
- joint caster_joint: origin xyz=0.1 0 -0.03 -> xyz=0.3 0 -0.09
- joint depth_camera_joint: origin xyz=0.155 0 0.02 rpy=0 0 0 -> xyz=0 0 0.25 rpy=0 0 0; parent base_link -> h_boom
- joint gps_joint: origin xyz=-0.1 0 0.025 -> xyz=-0.3 0 0.075
- joint imu_joint: origin xyz=0 0 0.025 -> xyz=0 0 0.075
- joint left_wheel_joint: origin xyz=0 0.12 0 rpy=-1.5708 0 0 -> xyz=0 0.36 0 rpy=-1.5708 0 0
- joint lidar_joint: origin xyz=0.1 0 0.035 -> xyz=0.3 0 0.105
- joint right_wheel_joint: origin xyz=0 -0.12 0 rpy=-1.5708 0 0 -> xyz=0 -0.36 0 rpy=-1.5708 0 0
